File: schematics/outlets/outlets.kicad_sch (KiCad schematic)
At the start: 3 parts, among them J1 Raspberry Pi, J2 5V Power Supply, K1 8 Channel Relay

Commit message: updated kicad version
Connections:
- net at K1. (VCC): now also J1.38 (GPIO20); no longer J2. (-)
- new net: J2. (-), K1. (VCC)
